File: PCB/HexaHubV2.kicad_sch (KiCad schematic)
At the start: 27 parts, among them J1 USB_C_Receptacle_USB2.0_16P, J2 USB_A, J3 USB_A, J4 USB_A, J5 USB_A, U1 SL2.1A, Y1 12MHz

Commit message: Slight changes to PCB and updated gerbers
Parts:
- F2, F3, F4, F5: value 2A -> 500mA
- renumbered C9 to C5, C10 to C6, C11 to C7, C12 to C8
Other:
- note added: "Downstream Ports"
- note added: "ESD Protection"
- note added: "Main IC"
- note added: "Upstream USB-C"
Changed lines of the file:
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@@
 	(generator_version "10.0")
 	(paper "A4")
+	(rectangle
+		(start 202.565 19.05)
+		(end 274.955 161.29)
+		(stroke
+			(width 0)
+			(type default)
+		)
+		(fill
+			(type none)
+		)
+	)
+	(rectangle
+		(start 19.05 17.78)
+		(end 116.84 73.025)
+		(stroke
+			(width 0)
+			(type default)
+		)
+		(fill
+			(type none)
+		)
+	)
+	(rectangle
+		(start 78.105 74.93)
+		(end 186.69 129.54)
+		(stroke
+			(width 0)
+			(type default)
+		)
+		(fill
+			(type none)
+		)
+	)
+	(rectangle
+		(start 15.24 136.525)
+		(end 175.26 194.945)
+		(stroke
+			(width 0)
+			(type default)
+		)
+		(fill
+			(type none)
+		)
+	)
+	(text "ESD Protection\n"
+		(exclude_from_sim no)
+		(at 157.734 192.532 0)
+		(effects
+			(font
+				(size 2.54 2.54)
+			)
+		)
+	)
+	(text "Main IC\n"
+		(exclude_from_sim no)
+		(at 86.106 127.762 0)
+		(effects
+			(font
+				(size 2.54 2.54)
+			)
+		)
+	)
+	(text "Downstream Ports\n"
+		(exclude_from_sim no)
+		(at 256.54 158.496 0)
+		(effects
+			(font
+				(size 2.54 2.54)
+			)
+		)
+	)
+	(text "Upstream USB-C\n"
+		(exclude_from_sim no)
+		(at 99.568 70.866 0)
+		(effects
+			(font
+				(size 2.54 2.54)
+			)
+		)
+	)
 	(junction
 		(at 218.44 115.57)
@@
 		(in_pos_files yes)
 		(dnp no)
-		(property "Reference" "C9"
+		(property "Reference" "C5"
 			(at 105.918 104.648 0)
 			(show_name no)
@@
 			(project "HexaHubV2"
 				(path "/9ae80488-f324-4720-8c95-5616f62f6793"
-					(reference "C9")
+					(reference "C5")
 					(unit 1)
 				)
@@
 			)
 		)
-		(property "Value" "2A"
+		(property "Value" "500mA"
 			(at 236.22 27.94 90)
 			(show_name no)
@@
 			)
 		)
-		(property "Value" "2A"
+		(property "Value" "500mA"
 			(at 234.95 97.79 90)
 			(show_name no)
@@
 			)
 		)
-		(property "Value" "2A"
+		(property "Value" "500mA"
 			(at 234.95 132.08 90)
 			(show_name no)
@@
 		(in_pos_files yes)
 		(dnp no)
-		(property "Reference" "C11"
+		(property "Reference" "C7"
 			(at 100.838 84.582 90)
 			(show_name no)
@@
 			(project "HexaHubV2"
 				(path "/9ae80488-f324-4720-8c95-5616f62f6793"
-					(reference "C11")
+					(reference "C7")
 					(unit 1)
 				)
@@
 		(in_pos_files yes)
 		(dnp no)
-		(property "Reference" "C10"
+		(property "Reference" "C6"
 			(at 97.028 104.648 0)
 			(show_name no)
@@
 			(project "HexaHubV2"
 				(path "/9ae80488-f324-4720-8c95-5616f62f6793"
-					(reference "C10")
+					(reference "C6")
 					(unit 1)
 				)
@@
 		(in_pos_files yes)
 		(dnp no)
-		(fields_autoplaced yes)
 		(property "Reference" "#PWR01"
 			(at 31.75 74.93 0)
@@
 		)
 		(property "Value" "GND"
-			(at 31.75 73.66 0)
+			(at 31.75 72.136 0)
 			(show_name no)
 			(do_not_autoplace no)
@@
 			)
 		)
-		(property "Value" "2A"
+		(property "Value" "500mA"
 			(at 236.22 63.5 90)
 			(show_name no)
@@
 		(in_pos_files yes)
 		(dnp no)
-		(property "Reference" "C12"
+		(property "Reference" "C8"
 			(at 100.584 92.202 90)
 			(show_name no)
@@
 			(project "HexaHubV2"
 				(path "/9ae80488-f324-4720-8c95-5616f62f6793"
-					(reference "C12")
+					(reference "C8")
 					(unit 1)
 				)
